File: PCB/MainBoard/MainBoard.kicad_pcb (KiCad board)
At the start: 2 copper layers, 306.8 x 129.6 mm, 170 parts, among them J1 Conn_01x04_12864, J2 Conn_02x20_Odd_Even, J3 Conn_01x03_Female, J4 Conn_01x04_12864, J5 Conn_01x03_Female, J6 Conn_01x04_12864, SW1 RotaryEncoder_Switch, SW10 SW_8, SW11 SW_9, SW12 SW_0, SW13 SW_-, SW14 SW_+, SW15 SW_esc, SW16 SW_tab, SW17 SW_q, SW18 SW_w, SW19 SW_e, SW2 SW_`, SW20 SW_r, SW21 SW_t, SW22 SW_y, SW23 SW_u, SW24 SW_i, SW25 SW_o, SW26 SW_p, SW27 SW_[, SW28 SW_back, SW29 SW_del, SW3 SW_1, SW30 SW_caps, SW31 SW_a, SW32 SW_s, SW33 SW_f, SW34 SW_g, SW35 SW_h, SW36 SW_j, SW37 SW_k, SW38 SW_l, SW39 SW_;, SW4 SW_2, SW40 SW_', SW41 SW_], SW42 SW_ins, SW43 SW_shift, SW44 SW_z, SW45 SW_x, SW46 SW_v, SW47 SW_b, SW48 SW_n, SW49 SW_m, SW5 SW_3, SW50 SW_,, SW51 SW_., SW52 SW_/, SW53 SW_r_shift, SW54 SW_\, SW55 SW_c, SW56 SW_fn1, SW57 SW_ctrl, SW58 SW_super, SW59 SW_alt, SW6 SW_4, SW60 SW_d, SW61 SW_space, SW62 SW_fn2, SW63 SW_left, SW64 SW_down, SW65 SW_up, SW66 SW_right, SW67 SW_enter, SW7 SW_5, SW8 SW_6, SW9 SW_7, U1 Pico

Commit message: Layout settled
Parts:
- removed the REF** at (291.9, 87.6)
- removed the REF** at (287.1, 106.7)
- removed the REF** at (294.2, 49.5)
- removed the REF** at (49.0, 106.7)
- added J8: JoyStick_Or_I2C1, Connector_JST:JST_PH_S4B-PH-K_1x04_P2.00mm_Horizontal, B.Cu at (131.0, 130.5)
- added REF**: Stabilizer_Cherry_MX_2.00u, Stabilizer_Cherry_MX_2.00u, F.Cu at (42.5, 106.7)
- added REF**: Stabilizer_Cherry_MX_2.00u, Stabilizer_Cherry_MX_2.00u, F.Cu at (287.8, 49.5)
- added REF**: Stabilizer_Cherry_MX_2.00u, Stabilizer_Cherry_MX_2.00u, F.Cu at (280.6, 106.7)
- added REF**: Stabilizer_Cherry_MX_2.00u, Stabilizer_Cherry_MX_2.00u, F.Cu at (285.4, 87.6)
- added SW68: SW_enter, PCM_Switch_Keyboard_Hotswap_Kailh:SW_Hotswap_Kailh_MX_2.25u, F.Cu at (285.4, 87.6)
- C1, C2: moved to B.Cu
- J1: value Conn_01x04_12864 -> PiPowerSwitch; footprint JMD0.96C:JMD0.96C -> Connector_PinHeader_2.54mm:PinHeader_1x03_P2.54mm_Vertical
- J2: value Conn_02x20_Odd_Even -> Pi_Zero
- J3: value Conn_01x03_Female -> I2C0; footprint Connector_PinHeader_2.54mm:PinHeader_1x03_P2.54mm_Vertical -> Connector_PinHeader_2.54mm:PinHeader_1x04_P2.54mm_Horizontal
- J4: value Conn_01x04_12864 -> JMD0.96C; footprint Connector_JST:JST_PH_S4B-PH-K_1x04_P2.00mm_Horizontal -> JMD0.96C:JMD0.96C; moved to F.Cu
- J5: value Conn_01x03_Female -> WS2812; footprint Connector_PinHeader_2.54mm:PinHeader_1x03_P2.54mm_Vertical -> Connector_PinHeader_2.54mm:PinHeader_1x03_P2.54mm_Horizontal
- J6: value Conn_01x04_12864 -> Extra_Keys
- SW1: value RotaryEncoder_Switch -> SPI_SW; footprint RotaryEncoder:RotaryEncoder_Alps_EC11E-Switch_Vertical_H20mm_CircularMountingHoles -> Button_Switch_THT:SW_DIP_SPSTx04_Slide_6.7x11.72mm_W7.62mm_P2.54mm_LowProfile
- SW10: value SW_8 -> SW_7
- SW11: value SW_9 -> SW_8
- SW12: value SW_0 -> SW_9
- SW13: value SW_- -> SW_0
- SW14: value SW_+ -> SW_-
- SW15: value SW_esc -> SW_+
- SW16: value SW_tab -> SW_esc; footprint PCM_Switch_Keyboard_Hotswap_Kailh:SW_Hotswap_Kailh_MX_1.50u -> PCM_Switch_Keyboard_Hotswap_Kailh:SW_Hotswap_Kailh_MX_1.00u
- SW17: value SW_q -> SW_tab; footprint PCM_Switch_Keyboard_Hotswap_Kailh:SW_Hotswap_Kailh_MX_1.00u -> PCM_Switch_Keyboard_Hotswap_Kailh:SW_Hotswap_Kailh_MX_1.50u
- SW18: value SW_w -> SW_q
- SW19: value SW_e -> SW_w
- SW2: value SW_` -> RotaryEncoder_Switch; footprint PCM_Switch_Keyboard_Hotswap_Kailh:SW_Hotswap_Kailh_MX_1.00u -> RotaryEncoder:RotaryEncoder_Alps_EC11E-Switch_Vertical_H20mm_CircularMountingHoles
- SW20: value SW_r -> SW_e
- SW21: value SW_t -> SW_r
- SW22: value SW_y -> SW_t
- SW23: value SW_u -> SW_y
- SW24: value SW_i -> SW_u
- SW25: value SW_o -> SW_i
- SW26: value SW_p -> SW_o
- SW27: value SW_[ -> SW_p
- SW28: value SW_back -> SW_[; footprint PCM_Switch_Keyboard_Hotswap_Kailh:SW_Hotswap_Kailh_MX_2.00u -> PCM_Switch_Keyboard_Hotswap_Kailh:SW_Hotswap_Kailh_MX_1.00u
- SW29: value SW_del -> SW_back; footprint PCM_Switch_Keyboard_Hotswap_Kailh:SW_Hotswap_Kailh_MX_1.00u -> PCM_Switch_Keyboard_Hotswap_Kailh:SW_Hotswap_Kailh_MX_2.00u
- SW3: value SW_1 -> SW_`
- SW30: value SW_caps -> SW_del; footprint PCM_Switch_Keyboard_Hotswap_Kailh:SW_Hotswap_Kailh_MX_1.75u -> PCM_Switch_Keyboard_Hotswap_Kailh:SW_Hotswap_Kailh_MX_1.00u
- SW31: value SW_a -> SW_caps; footprint PCM_Switch_Keyboard_Hotswap_Kailh:SW_Hotswap_Kailh_MX_1.00u -> PCM_Switch_Keyboard_Hotswap_Kailh:SW_Hotswap_Kailh_MX_1.75u
- SW32: value SW_s -> SW_a
- SW33: value SW_f -> SW_s
- SW34: value SW_g -> SW_f
- SW35: value SW_h -> SW_g
- SW36: value SW_j -> SW_h
- SW37: value SW_k -> SW_j
- SW38: value SW_l -> SW_k
- SW39: value SW_; -> SW_l
- SW4: value SW_2 -> SW_1
- SW40: value SW_' -> SW_;
- SW41: value SW_] -> SW_'
- SW42: value SW_ins -> SW_]
- SW43: value SW_shift -> SW_ins; footprint PCM_Switch_Keyboard_Hotswap_Kailh:SW_Hotswap_Kailh_MX_2.25u -> PCM_Switch_Keyboard_Hotswap_Kailh:SW_Hotswap_Kailh_MX_1.00u
- SW44: value SW_z -> SW_shift; footprint PCM_Switch_Keyboard_Hotswap_Kailh:SW_Hotswap_Kailh_MX_1.00u -> PCM_Switch_Keyboard_Hotswap_Kailh:SW_Hotswap_Kailh_MX_2.25u
- SW45: value SW_x -> SW_z
- SW46: value SW_v -> SW_x
- SW47: value SW_b -> SW_v
- SW48: value SW_n -> SW_b
- SW49: value SW_m -> SW_n
- SW5: value SW_3 -> SW_2
- SW50: value SW_, -> SW_m
- SW51: value SW_. -> SW_,
- SW52: value SW_/ -> SW_.
- SW53: value SW_r_shift -> SW_/; footprint PCM_Switch_Keyboard_Hotswap_Kailh:SW_Hotswap_Kailh_MX_2.75u -> PCM_Switch_Keyboard_Hotswap_Kailh:SW_Hotswap_Kailh_MX_1.00u
- SW54: value SW_\ -> SW_r_shift; footprint PCM_Switch_Keyboard_Hotswap_Kailh:SW_Hotswap_Kailh_MX_1.50u -> PCM_Switch_Keyboard_Hotswap_Kailh:SW_Hotswap_Kailh_MX_2.75u
- SW55: value SW_c -> SW_\; footprint PCM_Switch_Keyboard_Hotswap_Kailh:SW_Hotswap_Kailh_MX_1.00u -> PCM_Switch_Keyboard_Hotswap_Kailh:SW_Hotswap_Kailh_MX_1.50u
- SW56: value SW_fn1 -> SW_c
- SW57: value SW_ctrl -> SW_fn1; footprint PCM_Switch_Keyboard_Hotswap_Kailh:SW_Hotswap_Kailh_MX_1.25u -> PCM_Switch_Keyboard_Hotswap_Kailh:SW_Hotswap_Kailh_MX_1.00u
- SW58: value SW_super -> SW_ctrl
- SW59: value SW_alt -> SW_super
- SW6: value SW_4 -> SW_3
- SW60: value SW_d -> SW_alt; footprint PCM_Switch_Keyboard_Hotswap_Kailh:SW_Hotswap_Kailh_MX_1.00u -> PCM_Switch_Keyboard_Hotswap_Kailh:SW_Hotswap_Kailh_MX_1.25u
- SW61: value SW_space -> SW_d; footprint PCM_Switch_Keyboard_Hotswap_Kailh:SW_Hotswap_Kailh_MX_6.25u -> PCM_Switch_Keyboard_Hotswap_Kailh:SW_Hotswap_Kailh_MX_1.00u
- SW62: value SW_fn2 -> SW_space; footprint PCM_Switch_Keyboard_Hotswap_Kailh:SW_Hotswap_Kailh_MX_1.00u -> PCM_Switch_Keyboard_Hotswap_Kailh:SW_Hotswap_Kailh_MX_6.25u
- SW63: value SW_left -> SW_fn2
- SW64: value SW_down -> SW_left
- SW65: value SW_up -> SW_down
- SW66: value SW_right -> SW_up
- SW67: value SW_enter -> SW_right; footprint PCM_Switch_Keyboard_Hotswap_Kailh:SW_Hotswap_Kailh_MX_2.25u -> PCM_Switch_Keyboard_Hotswap_Kailh:SW_Hotswap_Kailh_MX_1.00u
- SW7: value SW_5 -> SW_4
- SW8: value SW_6 -> SW_5
- SW9: value SW_7 -> SW_6
- moved SW29 272.4 mm to (287.8, 49.5)
- moved SW42 253.6 mm to (268.7, 68.6)
- moved SW15 241.9 mm to (259.2, 49.5)
- moved SW1 193.2 mm to (203.6, 39.0), turned to 90 degrees
- moved SW55 178.6 mm to (292.5, 68.6)
- moved D71 146.3 mm to (85.9, 28.5), turned to 0 degrees
- moved J1 141.6 mm to (218.5, 35.0), turned to 90 degrees
- moved D1 136.1 mm to (85.9, 11.0), turned to 0 degrees
- moved D72 136.0 mm to (96.6, 28.5), turned to 0 degrees
- moved D2 125.1 mm to (96.6, 11.0), turned to 0 degrees
- moved J4 123.0 mm to (68.0, 23.0), turned to 0 degrees
- moved C2 116.5 mm to (41.3, 23.2), turned to 0 degrees
- moved D3 114.1 mm to (107.3, 11.0), turned to 0 degrees
- moved C1 113.6 mm to (41.3, 20.1), turned to 180 degrees
- moved D42 112.1 mm to (225.2, 18.0), turned to 0 degrees
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Connections:
- J1 pad 2: GND -> +5V
- J1 pad 3: I2C0_SCL -> /Pi_VCC
- J2 pad 2: +5V -> /Pi_VCC
- J2 pad 35: SPI_MISO -> PI_SPI_MISO
- J2 pad 36: SPI_CS -> PI_SPI_CS
- J2 pad 38: SPI_MOSI -> PI_SPI_MOSI
- J2 pad 4: +5V -> /Pi_VCC
- J2 pad 40: SPI_SCK -> PI_SPI_SCK
- J3 pad 1: +5V -> I2C0_SCL
- J3 pad 2: Net-(J3-Pin_2) -> I2C0_SDA
- J3 pad 3: GND -> +3V3
- J4 pad 1: ExtraSource -> +5V
- J4 pad 2: Extra1 -> GND
- J4 pad 3: Extra2 -> I2C0_SCL
- J4 pad 4: Extra3 -> I2C0_SDA
- J5 pad 1: Net-(J5-Pin_1) -> +5V
- J5 pad 2: GND -> Net-(J5-Pin_2)
- J5 pad 3: Net-(J5-Pin_3) -> GND
- J6 pad 1: +3V3 -> ExtraSource
- J6 pad 2: ANG1 -> Extra1
- J6 pad 3: ANG2 -> Extra2
- J6 pad 4: GND -> Extra3
- R1 pad 2: Net-(J3-Pin_2) -> Net-(J5-Pin_2)
- SW10 pad 1: Net-(D24-K) -> Net-(D23-K)
- SW10 pad 2: Net-(D10-A) -> Net-(D9-A)
- SW11 pad 1: Net-(D25-K) -> Net-(D24-K)
- SW11 pad 2: Net-(D11-A) -> Net-(D10-A)
- SW12 pad 1: Net-(D26-K) -> Net-(D25-K)
- SW12 pad 2: Net-(D12-A) -> Net-(D11-A)
- SW13 pad 1: Net-(D27-K) -> Net-(D26-K)
- SW13 pad 2: Net-(D13-A) -> Net-(D12-A)
- SW14 pad 1: Net-(D28-K) -> Net-(D27-K)
- SW14 pad 2: Net-(D14-A) -> Net-(D13-A)
- SW15 pad 1: Net-(D29-A) -> Net-(D28-K)
- SW15 pad 2: Encoder_SW_2 -> Net-(D14-A)
- SW16 pad 1: Net-(D30-A) -> Net-(D29-A)
- SW16 pad 2: Net-(D2-K) -> Encoder_SW_2
- SW17 pad 1: Net-(D31-A) -> Net-(D30-A)
- SW17 pad 2: Net-(D3-K) -> Net-(D2-K)
- SW18 pad 1: Net-(D32-A) -> Net-(D31-A)
- SW18 pad 2: Net-(D4-K) -> Net-(D3-K)
- SW19 pad 1: Net-(D33-A) -> Net-(D32-A)
- SW19 pad 2: ExtraSource -> Net-(D4-K)
- SW20 pad 1: Net-(D34-A) -> Net-(D33-A)
- SW20 pad 2: Net-(D6-K) -> ExtraSource
- SW21 pad 1: Net-(D35-A) -> Net-(D34-A)
- SW21 pad 2: Net-(D7-K) -> Net-(D6-K)
- SW22 pad 1: Net-(D36-K) -> Net-(D35-A)
- SW22 pad 2: Net-(D8-A) -> Net-(D7-K)
- SW23 pad 1: Net-(D37-K) -> Net-(D36-K)
- SW23 pad 2: Net-(D9-A) -> Net-(D8-A)
- SW24 pad 1: Net-(D38-K) -> Net-(D37-K)
- SW24 pad 2: Net-(D10-A) -> Net-(D9-A)
- SW25 pad 1: Net-(D39-K) -> Net-(D38-K)
- SW25 pad 2: Net-(D11-A) -> Net-(D10-A)
- SW26 pad 1: Net-(D40-K) -> Net-(D39-K)
- SW26 pad 2: Net-(D12-A) -> Net-(D11-A)
- SW27 pad 1: Net-(D41-K) -> Net-(D40-K)
- SW27 pad 2: Net-(D13-A) -> Net-(D12-A)
- SW28 pad 1: Net-(D42-K) -> Net-(D41-K)
- SW28 pad 2: Net-(D14-A) -> Net-(D13-A)
- SW29 pad 1: Net-(D43-A) -> Net-(D42-K)
- SW29 pad 2: Encoder_SW_2 -> Net-(D14-A)
- SW3 pad 1: Net-(D17-A) -> Net-(D16-A)
- SW3 pad 2: Net-(D3-K) -> Net-(D2-K)
- SW30 pad 1: Net-(D44-A) -> Net-(D43-A)
- SW30 pad 2: Net-(D2-K) -> Encoder_SW_2
- SW31 pad 1: Net-(D45-A) -> Net-(D44-A)
- SW31 pad 2: Net-(D3-K) -> Net-(D2-K)
- SW32 pad 1: Net-(D46-A) -> Net-(D45-A)
- SW32 pad 2: Net-(D4-K) -> Net-(D3-K)
- SW33 pad 1: Net-(D48-A) -> Net-(D46-A)
- SW33 pad 2: Net-(D6-K) -> Net-(D4-K)
- SW34 pad 1: Net-(D49-A) -> Net-(D48-A)
- SW34 pad 2: Net-(D7-K) -> Net-(D6-K)
- SW35 pad 1: Net-(D50-K) -> Net-(D49-A)
- SW35 pad 2: Net-(D8-A) -> Net-(D7-K)
- SW36 pad 1: Net-(D51-K) -> Net-(D50-K)
- SW36 pad 2: Net-(D9-A) -> Net-(D8-A)
- SW37 pad 1: Net-(D52-K) -> Net-(D51-K)
- SW37 pad 2: Net-(D10-A) -> Net-(D9-A)
- SW38 pad 1: Net-(D53-K) -> Net-(D52-K)
- SW38 pad 2: Net-(D11-A) -> Net-(D10-A)
- SW39 pad 1: Net-(D54-K) -> Net-(D53-K)
- SW39 pad 2: Net-(D12-A) -> Net-(D11-A)
- SW4 pad 1: Net-(D18-A) -> Net-(D17-A)
- SW4 pad 2: Net-(D4-K) -> Net-(D3-K)
- SW40 pad 1: Net-(D55-K) -> Net-(D54-K)
- SW40 pad 2: Net-(D13-A) -> Net-(D12-A)
- SW41 pad 1: Net-(D56-K) -> Net-(D55-K)
- SW41 pad 2: Net-(D14-A) -> Net-(D13-A)
- SW42 pad 1: Net-(D57-A) -> Net-(D56-K)
- SW42 pad 2: Encoder_SW_2 -> Net-(D14-A)
- SW43 pad 1: Net-(D58-A) -> Net-(D57-A)
- SW43 pad 2: Net-(D2-K) -> Encoder_SW_2
- SW44 pad 1: Net-(D59-A) -> Net-(D58-A)
- SW44 pad 2: Net-(D3-K) -> Net-(D2-K)
- SW45 pad 1: Net-(D60-A) -> Net-(D59-A)
- SW45 pad 2: Net-(D4-K) -> Net-(D3-K)
- SW46 pad 1: Net-(D62-A) -> Net-(D60-A)
- SW46 pad 2: Net-(D6-K) -> Net-(D4-K)
- SW47 pad 1: Net-(D63-A) -> Net-(D62-A)
- SW47 pad 2: Net-(D7-K) -> Net-(D6-K)
- SW48 pad 1: Net-(D64-K) -> Net-(D63-A)
- SW48 pad 2: Net-(D8-A) -> Net-(D7-K)
- SW49 pad 1: Net-(D65-K) -> Net-(D64-K)
- SW49 pad 2: Net-(D9-A) -> Net-(D8-A)
- SW5 pad 1: Net-(D19-A) -> Net-(D18-A)
- SW5 pad 2: ExtraSource -> Net-(D4-K)
- SW50 pad 1: Net-(D66-K) -> Net-(D65-K)
- SW50 pad 2: Net-(D10-A) -> Net-(D9-A)
- SW51 pad 1: Net-(D67-K) -> Net-(D66-K)
- SW51 pad 2: Net-(D11-A) -> Net-(D10-A)
- SW52 pad 1: Net-(D68-K) -> Net-(D67-K)
- SW52 pad 2: Net-(D12-A) -> Net-(D11-A)
- SW53 pad 1: Net-(D69-K) -> Net-(D68-K)
- SW53 pad 2: Net-(D13-A) -> Net-(D12-A)
- SW54 pad 1: Net-(D70-K) -> Net-(D69-K)
- SW54 pad 2: Net-(D14-A) -> Net-(D13-A)
- SW55 pad 1: unconnected-(SW55-A-Pad1) -> Net-(D70-K)
- SW55 pad 2: Net-(D6-K) -> Net-(D14-A)
- SW56 pad 1: Net-(D71-A) -> unconnected-(SW56-A-Pad1)
- SW56 pad 2: Encoder_SW_2 -> Net-(D6-K)
- SW57 pad 1: Net-(D72-A) -> Net-(D71-A)
- SW57 pad 2: Net-(D2-K) -> Encoder_SW_2
- SW58 pad 1: Net-(D73-A) -> Net-(D72-A)
- SW58 pad 2: Net-(D3-K) -> Net-(D2-K)
- SW59 pad 1: Net-(D74-A) -> Net-(D73-A)
- SW59 pad 2: Net-(D4-K) -> Net-(D3-K)
- SW6 pad 1: Net-(D20-A) -> Net-(D19-A)
- SW6 pad 2: Net-(D6-K) -> ExtraSource
- SW60 pad 1: Net-(D77-A) -> Net-(D74-A)
- SW60 pad 2: Net-(D7-K) -> Net-(D4-K)
- SW61 pad 1: Net-(D78-K) -> Net-(D77-A)
- SW61 pad 2: Net-(D8-A) -> Net-(D7-K)
- SW62 pad 1: Net-(D79-K) -> Net-(D78-K)
- SW62 pad 2: Net-(D9-A) -> Net-(D8-A)
- SW63 pad 1: Net-(D80-K) -> Net-(D79-K)
- SW63 pad 2: Net-(D10-A) -> Net-(D9-A)
- SW64 pad 1: Net-(D81-K) -> Net-(D80-K)
- SW64 pad 2: Net-(D11-A) -> Net-(D10-A)
- SW65 pad 1: Net-(D82-K) -> Net-(D81-K)
- SW65 pad 2: Net-(D12-A) -> Net-(D11-A)
- SW66 pad 1: Net-(D83-K) -> Net-(D82-K)
- SW66 pad 2: Net-(D13-A) -> Net-(D12-A)
- SW67 pad 1: Net-(D84-K) -> Net-(D83-K)
- SW67 pad 2: Net-(D14-A) -> Net-(D13-A)
- SW7 pad 1: Net-(D21-A) -> Net-(D20-A)
- SW7 pad 2: Net-(D7-K) -> Net-(D6-K)
- SW8 pad 1: Net-(D22-K) -> Net-(D21-A)
- SW8 pad 2: Net-(D8-A) -> Net-(D7-K)
- SW9 pad 1: Net-(D23-K) -> Net-(D22-K)
- SW9 pad 2: Net-(D9-A) -> Net-(D8-A)
- U1 pad 39: +5V -> unconnected-(U1-VSYS-Pad39)
- U1 pad 41: Net-(J5-Pin_3) -> unconnected-(U1-SWCLK-Pad41)
- U1 pad 42: GND -> unconnected-(U1-GND-Pad42)
- U1 pad 43: Net-(J5-Pin_1) -> unconnected-(U1-SWDIO-Pad43)
Other:
- board size 306.8 x 129.6 mm -> 308.8 x 130.2 mm

Commit message: Updated layout to add mounting holes
Parts:
- added REF**: MountingHole_3.2mm_M3, MountingHole:MountingHole_3.2mm_M3, F.Cu at (180.9, 34.9)
- added REF**: MountingHole_3.2mm_M3, MountingHole:MountingHole_3.2mm_M3, F.Cu at (260.5, 106.8)
- added REF**: MountingHole_3.2mm_M3, MountingHole_3.2mm_M3, F.Cu at (124.0, 121.7)
- added REF**: MountingHole_3.2mm_M3, MountingHole:MountingHole_3.2mm_M3, F.Cu at (3.40, 10.5)
- added REF**: MountingHole_3.2mm_M3, MountingHole:MountingHole_3.2mm_M3, F.Cu at (23.1, 68.1)
- added REF**: MountingHole_3.2mm_M3, MountingHole:MountingHole_3.2mm_M3, F.Cu at (93.0, 34.9)
- added REF**: MountingHole_3.2mm_M3, MountingHole:MountingHole_3.2mm_M3, F.Cu at (280.4, 68.1)
- added REF**: MountingHole_3.2mm_M3, MountingHole:MountingHole_3.2mm_M3, F.Cu at (163.9, 77.4)
- added REF**: MountingHole_3.2mm_M3, MountingHole_3.2mm_M3, F.Cu at (180.1, 121.7)
- added REF**: MountingHole_3.2mm_M3, MountingHole:MountingHole_3.2mm_M3, F.Cu at (23.2, 106.8)
- moved R5 53.7 mm to (159.0, 34.9), turned to 0 degrees
- moved R1 49.9 mm to (103.7, 34.9)
- moved R4 35.4 mm to (145.2, 34.9)
- moved R2 21.5 mm to (117.5, 34.9)
- moved R3 6.99 mm to (131.3, 34.9)
- moved J5 6.69 mm to (188.0, 37.5), turned to 0 degrees
- moved C2 4.14 mm to (41.4, 27.3), turned to 180 degrees
- moved SW1 4.03 mm to (207.6, 38.9)
- moved U1 4.00 mm to (26.0, 26.0)
- moved C1 3.89 mm to (41.4, 24.0)
- moved J1 3.53 mm to (222.1, 35.0)
Connections:
- R2 pad 1: Net-(R2-Pad1) -> Enc1
- R2 pad 2: Enc1 -> Net-(R2-Pad2)
- R3 pad 1: Net-(R2-Pad1) -> Net-(R2-Pad2)
- R4 pad 1: Net-(R4-Pad1) -> +3V3
- R4 pad 2: +3V3 -> Net-(R4-Pad2)
- R5 pad 1: Net-(R4-Pad1) -> Net-(R4-Pad2)
- SW2 pad A: Net-(R2-Pad1) -> Net-(R2-Pad2)
- SW2 pad B: Net-(R4-Pad1) -> Net-(R4-Pad2)
- U1 pad 12: R3 -> R2
- U1 pad 14: R4 -> R3
- U1 pad 15: R2 -> R4
- U1 pad 39: unconnected-(U1-VSYS-Pad39) -> +5V
Routing:
- net R1: track 0.00 -> 159.1 mm
- net R0: track 0.00 -> 159.1 mm

Commit message: Crazy wiring
Routing:
- net +5V: track 0.00 -> 230.5 mm, vias 0 -> 1
- net R2: track 0.00 -> 220.7 mm
- net R3: track 0.00 -> 214.2 mm
- net R4: track 0.00 -> 210.2 mm
- net Net-(D13-A): track 0.00 -> 153.6 mm, vias 0 -> 6
- net Net-(D12-A): track 0.00 -> 153.0 mm, vias 0 -> 2
- net Net-(D14-A): track 0.00 -> 148.3 mm
- net Net-(D82-K): track 0.00 -> 130.4 mm
- net Net-(D83-K): track 0.00 -> 128.4 mm
- net Net-(D9-A): track 0.00 -> 109.8 mm
- net Net-(D69-K): track 0.00 -> 109.1 mm
- net Net-(D10-A): track 0.00 -> 108.2 mm
- net Net-(D11-A): track 0.00 -> 108.2 mm
- net Net-(D7-K): track 0.00 -> 106.7 mm, vias 0 -> 2
- net Net-(D68-K): track 0.00 -> 99.4 mm
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