File: PCB/MainBoard/switch_matrix.kicad_sch (KiCad schematic)
At the start: 150 parts, among them SW10 SW_6, SW11 SW_7, SW12 SW_8, SW13 SW_9, SW14 SW_0, SW15 SW_-, SW16 SW_+, SW17 SW_esc, SW18 SW_tab, SW19 SW_q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

Commit message: Minor changes
Parts:
- SW56: value SW_\ -> SW_bkslash
Changed lines of the file:
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@@
       (effects (font (size 1.27 1.27)))
     )
-    (property "Value" "SW_\\" (at 257.81 111.76 0)
+    (property "Value" "SW_bkslash" (at 257.81 111.76 0)
       (effects (font (size 1.27 1.27)))
     )
